Commit message: iiwa urdf and detect button

File: iiwa_description/urdf/iiwa.gazebo.xacro (robot description, xacro)
@@ -18,4 +18,5 @@
       <plugin name="gazebo_ros_control" filename="libgazebo_ros_control.so">
         <robotNamespace>/${robot_name}</robotNamespace>
+        <legacyModeNS>true</legacyModeNS>
       </plugin>
     </gazebo>

File: iiwa_description/urdf/iiwa7.urdf (withenv).xacro (robot description, xacro)
@@ -13,5 +13,5 @@
   <link name="world"/>
   <joint name="world_base_joint" type="fixed">
-    <origin xyz="-0.63 -0.35 0.25" rpy="0 0 0"/>
+    <origin xyz="-0.63 -0.47 0.25" rpy="0 0 0"/>
     <parent link="world"/>
     <child link="base_link"/>
@@ -42,10 +42,10 @@
       <material name="Grey"/>
     </collision>
-    <!--self_collision_checking>
+    <self_collision_checking>
       <origin xyz="0 0 0" rpy="0 0 0"/>
       <geometry>
         <capsule radius="0.15" length="0.25"/>
       </geometry>
-    </self_collision_checking-->
+    </self_collision_checking>
   </link>
   <link name="base_link">
@@ -76,7 +76,24 @@
     </self_collision_checking>
   </link>
+  <gazebo reference="base_link">
+    <material>Gazebo/Grey</material>
+    <mu1>0.2</mu1>
+    <mu2>0.2</mu2>
+  </gazebo>
   <!--iiwa-->
   <xacro:iiwa7 hardware_interface="$(arg hardware_interface)" robot_name="$(arg robot_name)" parent="base_link">
-    <origin xyz="0.087 0.15 1.246" rpy="0 -1.5708 2.3562" />
+    <origin xyz="0.2056 0 0.58" rpy="0 0 ${1*PII/2}" />
   </xacro:iiwa7>
+    <!--iiwa-->
+  <xacro:iiwa7 hardware_interface="$(arg hardware_interface)" robot_name="right" parent="base_link">
+    <origin xyz="-0.2056 0 0.58" rpy="0 0 ${-1*PII/2}" />
+  </xacro:iiwa7>
+      <!-- Load Gazebo lib and set the robot namespace -->
+  <gazebo>
+    <plugin name="gazebo_ros_control" filename="libgazebo_ros_control.so">
+      <robotNamespace>/iiwa</robotNamespace>
+      <robotSimType>gazebo_ros_control/DefaultRobotHWSim</robotSimType>
+      <legacyModeNS>true</legacyModeNS>
+    </plugin>
+  </gazebo>
 </robot>

File: iiwa_description/urdf/iiwa7_MFTouch.xacro (robot description, xacro)
@@ -254,5 +254,5 @@
     <joint name="${robot_name}_joint_7" type="revolute">
       <parent link="${robot_name}_link_6"/>
-      <child link="${robot_name}_link_7"/>
+      <child link="${robot_name}_link_7_MFTouch"/>
       <origin xyz="0 0.081 0.06070" rpy="${- PI / 2} ${PI} 0"/>
       <axis xyz="0 0 1"/>
@@ -265,5 +265,5 @@
       <dynamics damping="${joint_damping}"/>
     </joint>
-    <link name="${robot_name}_link_7">
+    <link name="${robot_name}_link_7_MFTouch">
       <inertial>
         <origin xyz="0 0 0.02" rpy="0 0 0"/>
@@ -272,5 +272,5 @@
       </inertial>
       <visual>
-        <origin xyz="0 0 0" rpy="0 0 0"/>
+        <origin xyz="0 0 -0.0005" rpy="0 0 0"/>
         <geometry>
           <mesh filename="package://iiwa_description/meshes/iiwa7/visual/iiwa_MFTouch_m.stl"/>
@@ -279,5 +279,5 @@
       </visual>
       <collision>
-        <origin xyz="0 0 0" rpy="0 0 0"/>
+        <origin xyz="0 0 -0.0005" rpy="0 0 0"/>
         <geometry>
           <mesh filename="package://iiwa_description/meshes/iiwa7/collision/iiwa_MFTouch_m.stl"/>
@@ -286,145 +286,10 @@
       </collision>
     </link>
-    <joint name="${robot_name}_joint_8" type="fixed">
-      <parent link="${robot_name}_link_7"/>
-      <child link="${robot_name}_link_graspbase"/>
+    <joint name="${robot_name}_joint_ee" type="fixed">
+      <parent link="${robot_name}_link_7_MFTouch"/>
+      <child link="${robot_name}_link_ee"/>
       <origin xyz="0 0 0.071" rpy="0 0 0"/>
     </joint>
-    <link name="${robot_name}_link_graspbase">
-      <inertial>
-        <origin xyz="0 0 -0.025" rpy="0 0 0"/>
-        <mass value="0.001"/>
-        <inertia ixx="0.0001"  ixy="0"  ixz="0" iyy="0.0001" iyz="0" izz="0.0001" />
-      </inertial>
-      <visual>
-        <origin xyz="0 0 0" rpy="0 0 0"/>
-        <geometry>
-          <mesh filename="package://iiwa_description/meshes/iiwa7/visual/graspbase.STL"/>
-        </geometry>
-        <material name="Grey"/>
-      </visual>
-      <!--collision>
-        <origin xyz="0 0 0" rpy="0 0 0"/>
-        <geometry>
-          <mesh filename="package://iiwa_description/meshes/iiwa7/visual/graspbase.STL"/>
-        </geometry>
-        <material name="Grey"/>
-      </collision-->
-    </link>
-    <joint name="${robot_name}_joint_9" type="revolute">
-      <parent link="${robot_name}_link_graspbase"/>
-      <child link="${robot_name}_link_fingerbase"/>
-      <origin xyz="0.075 0 0.169" rpy="0 0 0"/>
-      <axis xyz="0 0 1"/>
-      <limit lower="${-175 * PI / 180}" upper="${175 * PI / 180}"
-             effort="${max_effort}" velocity="0.5" />
-      <safety_controller soft_lower_limit="${-173 * PI / 180}"
-                         soft_upper_limit="${173 * PI / 180}"
-                         k_position="${safety_controller_k_pos}"
-                         k_velocity="${safety_controller_k_vel}"/>
-      <dynamics damping="${joint_damping}"/>
-    </joint>
-    <link name="${robot_name}_link_fingerbase">
-      <inertial>
-        <origin xyz="0 0 0.0" rpy="0 0 0"/>
-        <mass value="0.1"/>
-        <inertia ixx="0.001"  ixy="0.0"  ixz="0" iyy="0.001" iyz="0" izz="0.001" />
-      </inertial>
-      <visual>
-        <origin xyz="0 0 0" rpy="0 0 0"/>
-        <geometry>
-          <mesh filename="package://iiwa_description/meshes/iiwa7/visual/fingerbase.STL"/>
-        </geometry>
-        <material name="Grey"/>
-      </visual>
-      <!--collision>
-        <origin xyz="0 0 0" rpy="0 0 0"/>
-        <geometry>
-          <mesh filename="package://iiwa_description/meshes/iiwa7/collision/fingerbase.STL"/>
-        </geometry>
-        <material name="Grey"/>
-      </collision-->
-    </link>
-    <joint name="${robot_name}_joint_10" type="prismatic">
-        <parent link="${robot_name}_link_fingerbase"/>
-        <child link="${robot_name}_link_finger1"/>
-        <origin xyz="0.0 -0.0105 0.024" rpy="0 0 0"/>
-        <axis xyz="0 1 0"/>
-        <limit lower="-0.007" upper="0.0105"
-               effort="${max_effort}" velocity="${max_velocity}" />
-        <safety_controller soft_lower_limit="-0.009"
-                           soft_upper_limit="0.0103"
-                           k_position="${safety_controller_k_pos}"
-                           k_velocity="${safety_controller_k_vel}"/>
-        <dynamics damping="${joint_damping}"/>
-    </joint>
-    <link name="${robot_name}_link_finger1">
-      <inertial>
-        <origin xyz="0 0 0.02" rpy="0 0 0"/>
-        <mass value="10"/>
-        <inertia ixx="0.001"  ixy="0.0"  ixz="0" iyy="0.001" iyz="0" izz="0.001" />
-      </inertial>
-      <visual>
-        <origin xyz="0 0 0" rpy="0 0 0"/>
-        <geometry>
-          <mesh filename="package://iiwa_description/meshes/iiwa7/visual/finger.STL"/>
-        </geometry>
-        <material name="Grey"/>
-      </visual>
-      <collision>
-        <origin xyz="0 0 0" rpy="0 0 0"/>
-        <geometry>
-          <mesh filename="package://iiwa_description/meshes/iiwa7/collision/finger.STL"/>
-        </geometry>
-        <material name="Grey"/>
-      </collision>
-    </link>
-    <joint name="${robot_name}_joint_11" type="prismatic">
-      <parent link="${robot_name}_link_fingerbase"/>
-      <child link="${robot_name}_link_finger2"/>
-      <origin xyz="0.0 0.0105 0.024" rpy="0 0 ${PI}"/>
-      <axis xyz="0 1 0"/>
-      <limit lower="-0.0105" upper="0.007"
-             effort="${max_effort}" velocity="${max_velocity}" />
-      <safety_controller soft_lower_limit="-0.0103"
-                         soft_upper_limit="0.005"
-                         k_position="${safety_controller_k_pos}"
-                         k_velocity="${safety_controller_k_vel}"/>
-      <dynamics damping="${joint_damping}"/>
-    </joint>
-    <link name="${robot_name}_link_finger2">
-      <inertial>
-        <origin xyz="0 0 0.02" rpy="0 0 0"/>
-        <mass value="10"/>
-        <inertia ixx="0.001"  ixy="0.0"  ixz="0" iyy="0.001" iyz="0" izz="0.001" />
-      </inertial>
-      <visual>
-        <origin xyz="0 0 0" rpy="0 0 0"/>
-        <geometry>
-          <mesh filename="package://iiwa_description/meshes/iiwa7/visual/finger.STL"/>
-        </geometry>
-        <material name="Grey"/>
-      </visual>
-      <collision>
-        <origin xyz="0 0 0" rpy="0 0 0"/>
-        <geometry>
-          <mesh filename="package://iiwa_description/meshes/iiwa7/collision/finger.STL"/>
-        </geometry>
-        <material name="Grey"/>
-      </collision>
-    </link>
-    <joint name="${robot_name}_joint_ee" type="fixed">
-      <parent link="${robot_name}_link_graspbase"/>
-      <child link="${robot_name}_link_ee"/>
-      <origin xyz="0.077 0 0.223" rpy="0 0 0"/>
-    </joint>
     <link name="${robot_name}_link_ee">
-    </link>
-    <joint name="${robot_name}_joint_camera" type="fixed">
-      <parent link="${robot_name}_link_graspbase"/>
-      <child link="${robot_name}_link_camera"/>
-      <origin xyz="0.077 0 0.223" rpy="0 ${-PI/2} 0"/>
-    </joint>
-    <link name="${robot_name}_link_camera">
     </link>
     <!--Extensions -->
